Commit message: Add instructions for adding a new robot in README

File: xacro/foot.xacro (robot description, xacro)
@@ -22,5 +22,5 @@
         <origin xyz="${xyz}" rpy="0 0 0"/>
         <geometry>
-          <mesh filename="file://@CMAKE_SOURCE_DIR@/xacro/meshes/foot.stl"/>
+          <mesh filename="file://@MESHES_DESTINATION@/foot.stl"/>
         </geometry>
         <material name="">
@@ -31,5 +31,5 @@
         <origin xyz="${xyz}" rpy="0 0 0"/>
         <geometry>
-          <mesh filename="file://@CMAKE_SOURCE_DIR@/xacro/meshes/foot.stl"/>
+          <mesh filename="file://@MESHES_DESTINATION@/foot.stl"/>
         </geometry>
       </collision>
