Commit message: adding a robot model 'doublepanda_default' consisting of two panda kinematic chains as a single robot

File: xacro/doublepanda_arm_default.urdf.xacro (robot description, xacro)
@@ -1,12 +1,16 @@
-<?xml version='1.0' encoding='utf-8'?>
+<?xml version="1.0" encoding="utf-8"?>
 <robot xmlns:xacro="http://www.ros.org/wiki/xacro" name="panda">
-	<xacro:arg name="gazebo" default="true"/>
-  <xacro:include filename="$(find franka_gazebo)/robots/panda_arm.xacro" >
-  	<xacro:arg name="gazebo" value="${gazebo}"/>
+  <xacro:arg name="gazebo" default="true"/>
+  <xacro:include filename="main.xacro">
+    <xacro:arg name="gazebo" value="${gazebo}"/>
   </xacro:include>
-  <xacro:include filename="@CMAKE_BINARY_DIR@/xacro/panda_armB.xacro" >
-  	<xacro:arg name="gazebo" value="${gazebo}"/>
+  <xacro:include filename="pandaA_arm.xacro">
+    <xacro:arg name="gazebo" value="${gazebo}"/>
   </xacro:include>
-  <xacro:panda_arm connected_to='world'/>
-  <xacro:panda_armB xyz="0.0 1 0" connected_to='panda_link8'/>
+  <xacro:include filename="pandaB_arm.xacro">
+    <xacro:arg name="gazebo" value="${gazebo}"/>
+  </xacro:include>
+  <xacro:main connected_to='world'/>
+  <xacro:panda_armA xyz="0 +1 0" connected_to='main_link'/>
+  <xacro:panda_armB xyz="0 -1 0" connected_to='main_link'/>
 </robot>

File: xacro/pandaA_arm.xacro (robot description, xacro)
@@ -1,10 +1,10 @@
 <?xml version='1.0' encoding='utf-8'?>
 <robot xmlns:xacro="http://www.ros.org/wiki/xacro" name="panda">
-  <xacro:macro name="panda_armB" params="arm_id:='panda' package_name:='franka_gazebo' connected_to:='' xyz:='0 0 0' rpy:='0 0 0'">
+  <xacro:macro name="panda_armA" params="arm_id:='panda' package_name:='franka_gazebo' connected_to:='' xyz:='0 0 0' rpy:='0 0 0'">
     <xacro:unless value="${not connected_to}">
-      <link name="${connected_to}"/>
-      <joint name="${arm_id}_joint_${connected_to}" type="fixed">
+      <!-- <link name="${connected_to}"/>-->
+      <joint name="${arm_id}_jointA_${connected_to}" type="fixed">
         <parent link="${connected_to}"/>
-        <child link="${arm_id}_linkB0"/>
+        <child link="${arm_id}_linkA0"/>
         <origin rpy="${rpy}" xyz="${xyz}"/>
       </joint>
@@ -13,7 +13,7 @@
     <xacro:if value="$(arg gazebo)">
       <!-- Gazebo Tags -->
-      <xacro:include filename="$(find franka_gazebo)/robots/panda_arm.gazebo.xacro"/>
+      <xacro:include filename="pandaA_arm.gazebo.xacro"/>
     </xacro:if>
-    <link name="${arm_id}_linkB0">
+    <link name="${arm_id}_linkA0">
       <inertial>
         <mass value="2.92" />
@@ -22,5 +22,5 @@
       </inertial>
       <visual>
-        <origin xyz="${xyz}" rpy="${rpy}"/>
+        <origin xyz="0 0 0" rpy="0 0 0"/>
         <geometry>
           <mesh filename="package://${package_name}/meshes/visual/link0.dae"/>
@@ -31,5 +31,5 @@
       </visual>
       <collision>
-        <origin xyz="${xyz}" rpy="${rpy}"/>
+        <origin xyz="0 0 0" rpy="0 0 0"/>
         <geometry>
           <mesh filename="package://${package_name}/meshes/collision/link0.stl"/>
@@ -37,5 +37,5 @@
       </collision>
     </link>
-    <link name="${arm_id}_linkB1">
+    <link name="${arm_id}_linkA1">
       <inertial>
         <mass value="2.74" />
@@ -44,5 +44,5 @@
       </inertial>
       <visual>
-        <origin xyz="${xyz}" rpy="${rpy}"/>
+        <origin xyz="0 0 0" rpy="0 0 0"/>
         <geometry>
           <mesh filename="package://${package_name}/meshes/visual/link1.dae"/>
@@ -53,5 +53,5 @@
       </visual>
       <collision>
-        <origin xyz="${xyz}" rpy="${rpy}"/>
+        <origin xyz="0 0 0" rpy="0 0 0"/>
         <geometry>
           <mesh filename="package://${package_name}/meshes/collision/link1.stl"/>
@@ -59,13 +59,13 @@
       </collision>
     </link>
-    <joint name="${arm_id}_jointB1" type="revolute">
+    <joint name="${arm_id}_jointA1" type="revolute">
       <safety_controller k_position="100.0" k_velocity="40.0" soft_lower_limit="-2.8973" soft_upper_limit="2.8973"/>
       <origin rpy="0 0 0" xyz="0 0 0.333"/>
-      <parent link="${arm_id}_linkB0"/>
-      <child link="${arm_id}_linkB1"/>
+      <parent link="${arm_id}_linkA0"/>
+      <child link="${arm_id}_linkA1"/>
       <axis xyz="0 0 1"/>
       <limit effort="87" lower="-2.8973" upper="2.8973" velocity="2.1750"/>
     </joint>
-    <link name="${arm_id}_linkB2">
+    <link name="${arm_id}_linkA2">
       <inertial>
         <mass value="2.74" />
@@ -74,5 +74,5 @@
       </inertial>
       <visual>
-        <origin xyz="${xyz}" rpy="${rpy}"/>
+        <origin xyz="0 0 0" rpy="0 0 0"/>
         <geometry>
           <mesh filename="package://${package_name}/meshes/visual/link2.dae"/>
@@ -83,5 +83,5 @@
       </visual>
       <collision>
-        <origin xyz="${xyz}" rpy="${rpy}"/>
+        <origin xyz="0 0 0" rpy="0 0 0"/>
         <geometry>
           <mesh filename="package://${package_name}/meshes/collision/link2.stl"/>
@@ -89,13 +89,13 @@
       </collision>
     </link>
-    <joint name="${arm_id}_jointB2" type="revolute">
+    <joint name="${arm_id}_jointA2" type="revolute">
       <safety_controller k_position="100.0" k_velocity="40.0" soft_lower_limit="-1.7628" soft_upper_limit="1.7628"/>
       <origin rpy="${-pi/2} 0 0" xyz="0 0 0"/>
-      <parent link="${arm_id}_linkB1"/>
-      <child link="${arm_id}_linkB2"/>
+      <parent link="${arm_id}_linkA1"/>
+      <child link="${arm_id}_linkA2"/>
       <axis xyz="0 0 1"/>
       <limit effort="87" lower="-1.7628" upper="1.7628" velocity="2.1750"/>
     </joint>
-    <link name="${arm_id}_linkB3">
+    <link name="${arm_id}_linkA3">
       <inertial>
         <mass value="2.38" />
@@ -104,5 +104,5 @@
       </inertial>
       <visual>
-        <origin xyz="${xyz}" rpy="${rpy}"/>
+        <origin xyz="0 0 0" rpy="0 0 0"/>
         <geometry>
           <mesh filename="package://${package_name}/meshes/visual/link3.dae"/>
@@ -113,5 +113,5 @@
       </visual>
       <collision>
-        <origin xyz="${xyz}" rpy="${rpy}"/>
+        <origin xyz="0 0 0" rpy="0 0 0"/>
         <geometry>
           <mesh filename="package://${package_name}/meshes/collision/link3.stl"/>
@@ -119,13 +119,13 @@
       </collision>
     </link>
-    <joint name="${arm_id}_jointB3" type="revolute">
+    <joint name="${arm_id}_jointA3" type="revolute">
       <safety_controller k_position="100.0" k_velocity="40.0" soft_lower_limit="-2.8973" soft_upper_limit="2.8973"/>
       <origin rpy="${pi/2} 0 0" xyz="0 -0.316 0"/>
-      <parent link="${arm_id}_linkB2"/>
-      <child link="${arm_id}_linkB3"/>
+      <parent link="${arm_id}_linkA2"/>
+      <child link="${arm_id}_linkA3"/>
       <axis xyz="0 0 1"/>
       <limit effort="87" lower="-2.8973" upper="2.8973" velocity="2.1750"/>
     </joint>
-    <link name="${arm_id}_linkB4">
+    <link name="${arm_id}_linkA4">
       <inertial>
         <mass value="2.38" />
@@ -134,5 +134,5 @@
       </inertial>
       <visual>
-        <origin xyz="${xyz}" rpy="${rpy}"/>
+        <origin xyz="0 0 0" rpy="0 0 0"/>
         <geometry>
           <mesh filename="package://${package_name}/meshes/visual/link4.dae"/>
@@ -143,5 +143,5 @@
       </visual>
       <collision>
-        <origin xyz="${xyz}" rpy="${rpy}"/>
+        <origin xyz="0 0 0" rpy="0 0 0"/>
         <geometry>
           <mesh filename="package://${package_name}/meshes/collision/link4.stl"/>
@@ -149,15 +149,15 @@
       </collision>
     </link>
-    <joint name="${arm_id}_jointB4" type="revolute">
+    <joint name="${arm_id}_jointA4" type="revolute">
       <safety_controller k_position="100.0" k_velocity="40.0" soft_lower_limit="-3.0718" soft_upper_limit="0.0698"/>
       <!-- soft_upper_limitr should be -0.0698, but that brakes simulation when initial position for this joint is 0.0 -->
       <origin rpy="${pi/2} 0 0" xyz="0.0825 0 0"/>
-      <parent link="${arm_id}_linkB3"/>
-      <child link="${arm_id}_linkB4"/>
+      <parent link="${arm_id}_linkA3"/>
+      <child link="${arm_id}_linkA4"/>
       <axis xyz="0 0 1"/>
       <limit effort="87" lower="-3.0718" upper="0.0698" velocity="2.1750"/>
       <!-- upper should be -0.0698, but that brakes simulation when initial position for this joint is 0.0 -->
     </joint>
-    <link name="${arm_id}_linkB5">
+    <link name="${arm_id}_linkA5">
       <inertial>
         <mass value="2.74" />
@@ -166,5 +166,5 @@
       </inertial>
       <visual>
-        <origin xyz="${xyz}" rpy="${rpy}"/>
+        <origin xyz="0 0 0" rpy="0 0 0"/>
         <geometry>
           <mesh filename="package://${package_name}/meshes/visual/link5.dae"/>
@@ -175,5 +175,5 @@
       </visual>
       <collision>
-        <origin xyz="${xyz}" rpy="${rpy}"/>
+        <origin xyz="0 0 0" rpy="0 0 0"/>
         <geometry>
           <mesh filename="package://${package_name}/meshes/collision/link5.stl"/>
@@ -181,13 +181,13 @@
       </collision>
     </link>
-    <joint name="${arm_id}_jointB5" type="revolute">
+    <joint name="${arm_id}_jointA5" type="revolute">
       <safety_controller k_position="100.0" k_velocity="40.0" soft_lower_limit="-2.8973" soft_upper_limit="2.8973"/>
       <origin rpy="${-pi/2} 0 0" xyz="-0.0825 0.384 0"/>
-      <parent link="${arm_id}_linkB4"/>
-      <child link="${arm_id}_linkB5"/>
+      <parent link="${arm_id}_linkA4"/>
+      <child link="${arm_id}_linkA5"/>
       <axis xyz="0 0 1"/>
       <limit effort="12" lower="-2.8973" upper="2.8973" velocity="2.6100"/>
     </joint>
-    <link name="${arm_id}_linkB6">
+    <link name="${arm_id}_linkA6">
       <inertial>
         <mass value="1.55" />
@@ -196,5 +196,5 @@
       </inertial>
       <visual>
-        <origin xyz="${xyz}" rpy="${rpy}"/>
+        <origin xyz="0 0 0" rpy="0 0 0"/>
         <geometry>
           <mesh filename="package://${package_name}/meshes/visual/link6.dae"/>
@@ -205,5 +205,5 @@
       </visual>
       <collision>
-        <origin xyz="${xyz}" rpy="${rpy}"/>
+        <origin xyz="0 0 0" rpy="0 0 0"/>
         <geometry>
           <mesh filename="package://${package_name}/meshes/collision/link6.stl"/>
@@ -211,13 +211,13 @@
       </collision>
     </link>
-    <joint name="${arm_id}_jointB6" type="revolute">
+    <joint name="${arm_id}_jointA6" type="revolute">
       <safety_controller k_position="100.0" k_velocity="40.0" soft_lower_limit="-0.0175" soft_upper_limit="3.7525"/>
       <origin rpy="${pi/2} 0 0" xyz="0 0 0"/>
-      <parent link="${arm_id}_linkB5"/>
-      <child link="${arm_id}_linkB6"/>
+      <parent link="${arm_id}_linkA5"/>
+      <child link="${arm_id}_linkA6"/>
       <axis xyz="0 0 1"/>
       <limit effort="12" lower="-0.0175" upper="3.7525" velocity="2.6100"/>
     </joint>
-    <link name="${arm_id}_link7">
+    <link name="${arm_id}_linkA7">
       <inertial>
         <mass value="0.54" />
@@ -226,5 +226,5 @@
       </inertial>
       <visual>
-        <origin xyz="${xyz}" rpy="${rpy}"/>
+        <origin xyz="0 0 0" rpy="0 0 0"/>
         <geometry>
           <mesh filename="package://${package_name}/meshes/visual/link7.dae"/>
@@ -235,5 +235,5 @@
       </visual>
       <collision>
-        <origin xyz="${xyz}" rpy="${rpy}"/>
+        <origin xyz="0 0 0" rpy="0 0 0"/>
         <geometry>
           <mesh filename="package://${package_name}/meshes/collision/link7.stl"/>
@@ -241,17 +241,17 @@
       </collision>
     </link>
-    <joint name="${arm_id}_jointB7" type="revolute">
+    <joint name="${arm_id}_jointA7" type="revolute">
       <safety_controller k_position="100.0" k_velocity="40.0" soft_lower_limit="-2.8973" soft_upper_limit="2.8973"/>
       <origin rpy="${pi/2} 0 0" xyz="0.088 0 0"/>
-      <parent link="${arm_id}_linkB6"/>
-      <child link="${arm_id}_linkB7"/>
+      <parent link="${arm_id}_linkA6"/>
+      <child link="${arm_id}_linkA7"/>
       <axis xyz="0 0 1"/>
       <limit effort="12" lower="-2.8973" upper="2.8973" velocity="2.6100"/>
     </joint>
-    <link name="${arm_id}_linkB8"/>
-    <joint name="${arm_id}_jointB8" type="fixed">
+    <link name="${arm_id}_linkA8"/>
+    <joint name="${arm_id}_jointA8" type="fixed">
       <origin rpy="0 0 0" xyz="0 0 0.107"/>
-      <parent link="${arm_id}_linkB7"/>
-      <child link="${arm_id}_linkB8"/>
+      <parent link="${arm_id}_linkA7"/>
+      <child link="${arm_id}_linkA8"/>
       <axis xyz="0 0 0"/>
     </joint>
