Commit message: fix joint limit for joint4, therefore generate single-panda in a similar manner as double-panda, see *.urdf.xacro files

File: xacro/pandaA_arm.xacro (robot description, xacro)
@@ -150,12 +150,10 @@
     </link>
     <joint name="${arm_id}_jointA4" type="revolute">
-      <safety_controller k_position="100.0" k_velocity="40.0" soft_lower_limit="-3.0718" soft_upper_limit="0.0698"/>
-      <!-- soft_upper_limitr should be -0.0698, but that brakes simulation when initial position for this joint is 0.0 -->
+      <safety_controller k_position="100.0" k_velocity="40.0" soft_lower_limit="-3.0718" soft_upper_limit="-0.0698"/>
       <origin rpy="${pi/2} 0 0" xyz="0.0825 0 0"/>
       <parent link="${arm_id}_linkA3"/>
       <child link="${arm_id}_linkA4"/>
       <axis xyz="0 0 1"/>
-      <limit effort="87" lower="-3.0718" upper="0.0698" velocity="2.1750"/>
-      <!-- upper should be -0.0698, but that brakes simulation when initial position for this joint is 0.0 -->
+      <limit effort="87" lower="-3.0718" upper="-0.0698" velocity="2.1750"/>
     </joint>
     <link name="${arm_id}_linkA5">

File: xacro/pandaB_arm.xacro (robot description, xacro)
@@ -150,12 +150,10 @@
     </link>
     <joint name="${arm_id}_jointB4" type="revolute">
-      <safety_controller k_position="100.0" k_velocity="40.0" soft_lower_limit="-3.0718" soft_upper_limit="0.0698"/>
-      <!-- soft_upper_limitr should be -0.0698, but that brakes simulation when initial position for this joint is 0.0 -->
+      <safety_controller k_position="100.0" k_velocity="40.0" soft_lower_limit="-3.0718" soft_upper_limit="-0.0698"/>
       <origin rpy="${pi/2} 0 0" xyz="0.0825 0 0"/>
       <parent link="${arm_id}_linkB3"/>
       <child link="${arm_id}_linkB4"/>
       <axis xyz="0 0 1"/>
-      <limit effort="87" lower="-3.0718" upper="0.0698" velocity="2.1750"/>
-      <!-- upper should be -0.0698, but that brakes simulation when initial position for this joint is 0.0 -->
+      <limit effort="87" lower="-3.0718" upper="-0.0698" velocity="2.1750"/>
     </joint>
     <link name="${arm_id}_linkB5">

File: xacro/panda_arm_default.urdf.xacro (robot description, xacro)
@@ -8,9 +8,5 @@
     <xacro:arg name="gazebo" value="${gazebo}"/>
   </xacro:include>
-  <xacro:include filename="@CMAKE_BINARY_DIR@/xacro/pandaB_arm.xacro">
-    <xacro:arg name="gazebo" value="${gazebo}"/>
-  </xacro:include>
   <xacro:main connected_to='world'/>
-  <xacro:panda_armA xyz="0 +1 0" connected_to='main_link'/>
-  <xacro:panda_armB xyz="0 -1 0" connected_to='main_link'/>
+  <xacro:panda_armA xyz="0 0 0" connected_to='main_link'/>
 </robot>

File: xacro/panda_arm_foot.urdf.xacro (robot description, xacro)
@@ -2,9 +2,13 @@
 <robot xmlns:xacro="http://www.ros.org/wiki/xacro" name="panda">
   <xacro:arg name="gazebo" default="true"/>
-  <xacro:include filename="$(find franka_gazebo)/robots/panda_arm.xacro">
+  <xacro:include filename="@CMAKE_BINARY_DIR@/xacro/main.xacro">
+    <xacro:arg name="gazebo" value="${gazebo}"/>
+  </xacro:include>
+  <xacro:include filename="@CMAKE_BINARY_DIR@/xacro/pandaA_arm.xacro">
     <xacro:arg name="gazebo" value="${gazebo}"/>
   </xacro:include>
   <xacro:include filename="@CMAKE_BINARY_DIR@/xacro/foot.xacro"/>
-  <xacro:panda_arm connected_to='world'/>
-  <xacro:foot ns="panda" rpy="0 0 ${-pi/4}" connected_to="panda_link8"/>
+  <xacro:main connected_to='world'/>
+  <xacro:panda_armA xyz="0 0 0" connected_to='main_link'/>
+  <xacro:foot ns="panda" rpy="0 0 ${-pi/4}" connected_to="panda_linkA8"/>
 </robot>

File: xacro/panda_arm_hand.urdf.xacro (robot description, xacro)
@@ -8,9 +8,7 @@
     <xacro:arg name="gazebo" value="${gazebo}"/>
   </xacro:include>
-  <xacro:include filename="@CMAKE_BINARY_DIR@/xacro/pandaB_arm.xacro">
-    <xacro:arg name="gazebo" value="${gazebo}"/>
-  </xacro:include>
+  <xacro:include filename="$(find franka_gazebo)/robots/hand.xacro"/>
   <xacro:main connected_to='world'/>
-  <xacro:panda_armA xyz="0 +1 0" connected_to='main_link'/>
-  <xacro:panda_armB xyz="0 -1 0" connected_to='main_link'/>
+  <xacro:panda_armA xyz="0 0 0" connected_to='main_link'/>
+  <xacro:hand ns="panda" rpy="0 0 ${-pi/4}" connected_to="panda_linkA8"/>
 </robot>
